Commit message: Finished part 1.

File: diff_drive/urdf/ddrive.gazebo.xacro (robot description, xacro)
@@ -6,6 +6,6 @@
   </gazebo>
   <gazebo reference="left_wheel">
-    <mu1>0.1</mu1>
-    <mu2>0.1</mu2>
+    <mu1>1000</mu1>
+    <mu2>9999</mu2>
     <minDepth>0.001</minDepth>
     <fdir1>1 0 0</fdir1>
@@ -16,6 +16,6 @@
   </gazebo>
   <gazebo reference="right_wheel">
-    <mu1>0.1</mu1>
-    <mu2>0.1</mu2>
+    <mu1>1000</mu1>
+    <mu2>9999</mu2>
     <minDepth>0.001</minDepth>
     <fdir1>1 0 0</fdir1>

File: diff_drive/urdf/ddrive.urdf.xacro (robot description, xacro)
@@ -23,9 +23,4 @@
     <color rgba="0 0 0 1"/>
   </material>
-  <!-- <link name="world"/>
-  <joint name="fixed" type="fixed">
-    <parent link="world"/>
-    <child link="base_link"/>
-  </joint> -->
   <link name="base_link">
     <visual>
